Commit message: simple robot

File: project_ws/install/telerobot_description/share/telerobot_description/urdf/camera.xacro (robot description, xacro)
@@ -1,47 +1 @@
-<?xml version="1.0"?>
-<robot xmlns:xacro="http://www.ros.org/wiki/xacro">
-    <xacro:property name="camera_length" value="0.01" />
-    <xacro:property name="camera_width" value="0.1" />
-    <xacro:property name="camera_height" value="0.05" />
-    <link name="camera_link">
-        <visual>
-            <geometry>
-                <box size="${camera_length} ${camera_width} ${camera_height}" />
-            </geometry>
-            <material name="grey" />
-        </visual>
-        <collision>
-            <geometry>
-                <box size="${camera_length} ${camera_width} ${camera_height}" />
-            </geometry>
-        </collision>
-        <xacro:box_inertia m="0.1" l="${camera_length}" w="${camera_width}" h="${camera_height}"
-                           xyz="0 0 0" rpy="0 0 0" />
-    </link>
-    <joint name="base_camera_joint" type="fixed">
-        <parent link="tower_link" />
-        <child link="camera_link" />
-        <origin xyz="${(tower_width + camera_length) / 2.0} 0 ${tower_height * 0.8}" rpy="0 0 0" />
-    </joint>
-    <link name="camera_link_optical">
-    </link>
-    <joint name="camera_optical_joint" type="fixed">
-        <!-- these values have to be these values otherwise the gazebo camera
-            image won't be aligned properly with the frame it is supposedly
-            originating from -->
-        <origin xyz="0 0 0" rpy="${-pi/2} 0 ${-pi/2}"/>
-        <parent link="camera_link"/>
-        <child link="camera_link_optical"/>
-    </joint>
-    <gazebo reference="camera_link">
-        <material>Gazebo/Red</material>
-        <sensor name="camera_sensor" type="camera">
-            <pose>0 0 0 0 0 0</pose>
-            <visualize>true</visualize>
-            <update_rate>10.0</update_rate>
-            <plugin name="camera_controller" filename="libgazebo_ros_camera.so">
-                <frame_name>camera_link_optical</frame_name>
-            </plugin>
-        </sensor>
-    </gazebo>
-</robot>
+/media/ros/fedora/home/maylis/Dokumente/TeleNav/project_ws/src/telerobot_description/urdf/camera.xacro

File: project_ws/install/telerobot_description/share/telerobot_description/urdf/common_properties.xacro (robot description, xacro)
@@ -1,39 +1 @@
-<?xml version="1.0"?>
-<robot xmlns:xacro="http://www.ros.org/wiki/xacro">
-    <material name="blue">
-        <color rgba="0 0 0.5 1" />
-    </material>
-    <material name="grey">
-        <color rgba="0.5 0.5 0.5 1" />
-    </material>
-    <material name="red">
-        <color rgba="0.5 0 0 1" />
-    </material>
-    <xacro:macro name="box_inertia" params="m l w h xyz rpy">
-        <inertial>
-            <origin xyz="${xyz}" rpy="${rpy}" />
-            <mass value="${m}" />
-            <inertia ixx="${(m/12) * (h*h + l*l)}" ixy="0" ixz="0"
-                     iyy="${(m/12) * (w*w + l*l)}" iyz="0"
-                     izz="${(m/12) * (w*w + h*h)}" />
-        </inertial>
-    </xacro:macro>
-    <xacro:macro name="cylinder_inertia" params="m r h xyz rpy">
-        <inertial>
-            <origin xyz="${xyz}" rpy="${rpy}" />
-            <mass value="${m}" />
-            <inertia ixx="${(m/12) * (3*r*r + h*h)}" ixy="0" ixz="0"
-                     iyy="${(m/12) * (3*r*r + h*h)}" iyz="0"
-                     izz="${(m/2) * (r*r)}" />
-        </inertial>
-    </xacro:macro>
-    <xacro:macro name="sphere_inertia" params="m r xyz rpy">
-        <inertial>
-            <origin xyz="${xyz}" rpy="${rpy}" />
-            <mass value="${m}" />
-            <inertia ixx="${(2/5) * m * r * r}" ixy="0" ixz="0"
-                     iyy="${(2/5) * m * r * r}" iyz="0"
-                     izz="${(2/5) * m * r * r}" />
-        </inertial>
-    </xacro:macro>
-</robot>
+/media/ros/fedora/home/maylis/Dokumente/TeleNav/project_ws/src/telerobot_description/urdf/common_properties.xacro

File: project_ws/install/telerobot_description/share/telerobot_description/urdf/lidar.xacro (robot description, xacro)
@@ -1,66 +1 @@
-<?xml version="1.0"?>
-<robot xmlns:xacro="http://www.ros.org/wiki/xacro">
-    <!-- Corrected property names and more reasonable dimensions -->
-    <xacro:property name="lidar_radius" value="0.05" />
-    <xacro:property name="lidar_length" value="0.05" />
-    <!-- Macro for cylinder inertia (if not already defined elsewhere) -->
-    <xacro:macro name="cylinder_inertia" params="m r h xyz rpy">
-        <inertial>
-            <origin xyz="${xyz}" rpy="${rpy}" />
-            <mass value="${m}" />
-            <inertia ixx="${m*(3*r*r + h*h)/12}" ixy="0" ixz="0"
-                     iyy="${m*(3*r*r + h*h)/12}" iyz="0"
-                     izz="${m*r*r/2}" />
-        </inertial>
-    </xacro:macro>
-    <link name="lidar_link">
-        <visual>
-            <geometry>
-                <cylinder radius="${lidar_radius}" length="${lidar_length}"/>
-            </geometry>
-            <material name="grey" />
-        </visual>
-        <collision>
-            <geometry>
-                <cylinder radius="${lidar_radius}" length="${lidar_length}"/>
-            </geometry>
-        </collision>
-        <xacro:cylinder_inertia m="0.1" r="${lidar_radius}" h="${lidar_length}"
-                           xyz="0 0 0" rpy="0 0 0" />
-    </link>
-    <joint name="base_lidar_joint" type="fixed">
-        <parent link="tower_link" />
-        <child link="lidar_link" />
-        <!-- Placing lidar on top of the base (base_height is 0.2) -->
-        <origin xyz="0 0 ${tower_height+0.01}" rpy="0 0 0" />
-    </joint>
-    <gazebo reference="lidar_link">
-        <material>Gazebo/Red</material>
-        <sensor name="laser" type="ray">
-            <pose>0 0 0 0 0 0</pose>
-            <visualize>true</visualize>
-            <update_rate>10.0</update_rate>
-            <ray>
-                <scan>
-                    <horizontal>
-                        <samples>360</samples>
-                        <min_angle>-3.14</min_angle>
-                        <max_angle>3.14</max_angle>
-                    </horizontal>
-                </scan>
-                <range>
-                    <min>0.3</min>
-                    <max>12</max>
-                </range>
-            </ray>
-            <plugin name="laser_controller" filename="libgazebo_ros_ray_sensor.so">
-                <ros>
-                    <argument>--remap ~/out:=scan</argument>
-                </ros>
-                <output_type>sensor_msgs/LaserScan</output_type>
-                <!-- Changed to match link name -->
-                <frame_name>lidar_link</frame_name>
-            </plugin>
-        </sensor>
-    </gazebo>
-</robot>
+/media/ros/fedora/home/maylis/Dokumente/TeleNav/project_ws/src/telerobot_description/urdf/lidar.xacro

File: project_ws/install/telerobot_description/share/telerobot_description/urdf/my_robot.urdf.xacro (robot description, xacro)
@@ -1,10 +1 @@
-<?xml version="1.0"?>
-<robot name="my_robot" xmlns:xacro="http://www.ros.org/wiki/xacro">
-    <!-- Robot Base-->
-    <xacro:include filename="common_properties.xacro" />
-    <xacro:include filename="robot_base.xacro" />
-    <xacro:include filename="robot_base_gazebo.xacro" />
-    <!-- Sensors-->
-     <xacro:include filename="camera.xacro"/>
-     <xacro:include filename="lidar.xacro"/>
-</robot>
+/media/ros/fedora/home/maylis/Dokumente/TeleNav/project_ws/src/telerobot_description/urdf/my_robot.urdf.xacro

File: project_ws/install/telerobot_description/share/telerobot_description/urdf/robot_base.xacro (robot description, xacro)
@@ -1,157 +1 @@
-<?xml version="1.0"?>
-<robot xmlns:xacro="http://www.ros.org/wiki/xacro">
-    <!-- Robot Base-->
-    <xacro:property name="base_length" value="0.6" />
-    <xacro:property name="base_width" value="0.6" />
-    <xacro:property name="base_height" value="0.2" />
-    <xacro:property name="wheel_radius" value="0.1" />
-    <xacro:property name="wheel_length" value="0.05" />
-    <!-- tower-->
-    <xacro:property name="tower_length" value="0.3" />
-    <xacro:property name="tower_width" value="0.3" />
-    <xacro:property name="tower_height" value="1.0" />
-    <link name="base_footprint" />
-    <link name="base_link">
-        <visual>
-            <geometry>
-                <box size="${base_length} ${base_width} ${base_height}" />
-            </geometry>
-            <origin xyz="0 0 ${base_height / 2.0}" rpy="0 0 0" />
-            <material name="blue" />
-        </visual>
-        <collision>
-            <geometry>
-                <box size="${base_length} ${base_width} ${base_height}" />
-            </geometry>
-            <origin xyz="0 0 ${base_height / 2.0}" rpy="0 0 0" />
-        </collision>
-        <xacro:box_inertia m="5.0" l="${2*base_length}" w="${2*base_width}" h="${2*base_height}"
-                           xyz="0 0 ${base_height / 2.0}" rpy="0 0 0" />
-    </link>
-    <link name="front_bumper_link">
-        <visual>
-            <geometry>
-                <cylinder radius="${base_width/2}" length="${base_height}"/>
-            </geometry>
-            <origin xyz="0 0 ${base_height / 2.0}" rpy="0 0 0" />
-            <material name="blue" />
-        </visual>
-        <collision>
-            <geometry>
-                <box size="${base_width} ${base_width} ${base_height}" />
-            </geometry>
-            <origin xyz="0 0 ${base_height / 2.0}" rpy="0 0 0" />
-        </collision>
-        <xacro:cylinder_inertia m="5.0" r="${base_width/2}" h="${base_width}"
-                           xyz="0 0 ${base_width / 2.0}" rpy="0 0 0" />
-    </link>
-    <link name="back_bumper_link">
-        <visual>
-            <geometry>
-                <cylinder radius="${base_width/2}" length="${base_height}"/>
-            </geometry>
-            <origin xyz="0 0 ${base_height / 2.0}" rpy="0 0 0" />
-            <material name="blue" />
-        </visual>
-        <collision>
-            <geometry>
-                <box size="${base_width} ${base_width} ${base_height}" />
-            </geometry>
-            <origin xyz="0 0 ${base_height / 2.0}" rpy="0 0 0" />
-        </collision>
-        <xacro:cylinder_inertia m="5.0" r="${base_width/2}" h="${base_width}"
-                           xyz="0 0 ${base_width / 2.0}" rpy="0 0 0" />
-    </link>
-    <link name="tower_link">
-        <visual>
-            <geometry>
-                <box size="${tower_length} ${tower_width} ${tower_height}" />
-            </geometry>
-            <origin xyz="0 0 ${tower_height/2.0}" rpy="0 0 0" />
-            <material name="blue" />
-        </visual>
-        <collision>
-            <geometry>
-                <box size="${tower_length} ${tower_width} ${tower_height}" />
-            </geometry>
-            <origin xyz="0 0 ${tower_height}" rpy="0 0 0" />
-        </collision>
-        <xacro:box_inertia m="5.0" l="${2*tower_length}" w="${2*tower_width}" h="${2*tower_height}"
-                           xyz="0 0 ${tower_height / 2.0}" rpy="0 0 0" />
-    </link>
-    <xacro:macro name="wheel_link" params="prefix">
-        <link name="${prefix}_wheel_link">
-            <visual>
-                <geometry>
-                    <cylinder radius="${wheel_radius}" length="${wheel_length}" />
-                </geometry>
-                <origin xyz="0 0 0" rpy="${pi / 2.0} 0 0" />
-                <material name="grey" />
-            </visual>
-            <collision>
-                <geometry>
-                    <cylinder radius="${wheel_radius}" length="${wheel_length}" />
-                </geometry>
-                <origin xyz="0 0 0" rpy="${pi / 2.0} 0 0" />
-            </collision>
-            <xacro:cylinder_inertia m="1.0" r="${2*wheel_radius}" h="${2*wheel_length}"
-                                    xyz="0 0 0" rpy="${pi / 2.0} 0 0" />
-        </link>
-    </xacro:macro>
-    <xacro:wheel_link prefix="right" />
-    <xacro:wheel_link prefix="left" />
-    <link name="caster_wheel_link">
-        <visual>
-            <geometry>
-                <sphere radius="${wheel_radius / 2.0}" />
-            </geometry>
-            <origin xyz="0 0 0" rpy="0 0 0" />
-            <material name="grey" />
-        </visual>
-        <collision>
-            <geometry>
-                <sphere radius="${wheel_radius / 2.0}" />
-            </geometry>
-            <origin xyz="0 0 0" rpy="0 0 0" />
-        </collision>
-        <xacro:sphere_inertia m="0.5" r="${2*wheel_radius / 2.0}"
-                              xyz="0 0 0" rpy="0 0 0" />
-    </link>
-    <joint name="front_bumper_joint" type="fixed">
-        <parent link="base_link" />
-        <child link="front_bumper_link" />
-        <origin xyz="${base_length / 2.0} 0 0" rpy="0 0 0" />
-    </joint>
-    <joint name="back_bumper_joint" type="fixed">
-        <parent link="base_link" />
-        <child link="back_bumper_link" />
-        <origin xyz="${-base_length / 2.0} 0 0" rpy="0 0 0" />
-    </joint>
-    <joint name="base_joint" type="fixed">
-        <parent link="base_footprint" />
-        <child link="base_link" />
-        <origin xyz="0 0 ${wheel_radius}" rpy="0 0 0"/>
-    </joint>
-    <joint name="tower_joint" type="fixed">
-        <parent link="base_link" />
-        <child link="tower_link" />
-        <origin xyz="0 0 ${base_height}" rpy="0 0 0" />
-    </joint>
-    <joint name="base_right_wheel_joint" type="continuous">
-        <parent link="base_link" />
-        <child link="right_wheel_link" />
-        <origin xyz="${-base_length / 4.0} ${-(base_width + wheel_length) / 2.0} 0" rpy="0 0 0" />
-        <axis xyz="0 1 0" />
-    </joint>
-    <joint name="base_left_wheel_joint" type="continuous">
-        <parent link="base_link" />
-        <child link="left_wheel_link" />
-        <origin xyz="${-base_length / 4.0} ${(base_width + wheel_length) / 2.0} 0" rpy="0 0 0" />
-        <axis xyz="0 1 0" />
-    </joint>
-    <joint name="base_caster_wheel_joint" type="fixed">
-        <parent link="base_link" />
-        <child link="caster_wheel_link" />
-        <origin xyz="${base_length / 3.0} 0 ${-wheel_radius / 2.0}" rpy="0 0 0" />
-    </joint>
-</robot>
+/media/ros/fedora/home/maylis/Dokumente/TeleNav/project_ws/src/telerobot_description/urdf/robot_base.xacro

File: project_ws/install/telerobot_description/share/telerobot_description/urdf/robot_base_gazebo.xacro (robot description, xacro)
@@ -1,26 +1 @@
-ä<?xml version="1.0"?>
-<robot xmlns:xacro="http://www.ros.org/wiki/xacro"
-      xmlns:ros_gz_sim="http://gazebosim.org/schema/ros_gz_sim">
-    <gazebo reference="caster_wheel_link">
-        <mu1 value="0.1" />
-        <mu2 value="0.1" />
-    </gazebo>
-    <gazebo>
-        <plugin filename="gz-sim-diff-drive-system"
-                name="gz::sim::systems::DiffDrive">
-            <left_joint>base_left_wheel_joint</left_joint>
-            <right_joint>base_right_wheel_joint</right_joint>
-            <wheel_separation>0.45</wheel_separation>
-            <wheel_radius>0.1</wheel_radius>
-            <frame_id>odom</frame_id>
-            <child_frame_id>base_footprint</child_frame_id>
-        </plugin>
-    </gazebo>
-    <gazebo>
-        <plugin filename="libignition-gazebo6-joint-state-publisher-system"
-                name="gz::sim::systems::JointStatePublisher">
-            <joint_name>base_left_wheel_joint</joint_name>
-            <joint_name>base_right_wheel_joint</joint_name>
-        </plugin>
-    </gazebo>
-</robot>
+/media/ros/fedora/home/maylis/Dokumente/TeleNav/project_ws/src/telerobot_description/urdf/robot_base_gazebo.xacro

File: project_ws/src/telerobot_description/urdf/lidar.xacro (robot description, xacro)
@@ -4,14 +4,4 @@
     <xacro:property name="lidar_radius" value="0.05" />
     <xacro:property name="lidar_length" value="0.05" />
-    <!-- Macro for cylinder inertia (if not already defined elsewhere) -->
-    <xacro:macro name="cylinder_inertia" params="m r h xyz rpy">
-        <inertial>
-            <origin xyz="${xyz}" rpy="${rpy}" />
-            <mass value="${m}" />
-            <inertia ixx="${m*(3*r*r + h*h)/12}" ixy="0" ixz="0"
-                     iyy="${m*(3*r*r + h*h)/12}" iyz="0"
-                     izz="${m*r*r/2}" />
-        </inertial>
-    </xacro:macro>
     <link name="lidar_link">
         <visual>
@@ -36,28 +26,31 @@
     </joint>
     <gazebo reference="lidar_link">
-        <material>Gazebo/Red</material>
-        <sensor name="laser" type="ray">
-            <pose>0 0 0 0 0 0</pose>
+        <sensor name="lidar" type="ray">
+            <always_on>true</always_on>
             <visualize>true</visualize>
-            <update_rate>10.0</update_rate>
+            <update_rate>5</update_rate>
             <ray>
-                <scan>
-                    <horizontal>
-                        <samples>360</samples>
-                        <min_angle>-3.14</min_angle>
-                        <max_angle>3.14</max_angle>
-                    </horizontal>
-                </scan>
-                <range>
-                    <min>0.3</min>
-                    <max>12</max>
-                </range>
+            <scan>
+                <horizontal>
+                <samples>360</samples>
+                <resolution>1.000000</resolution>
+                <min_angle>0.000000</min_angle>
+                <max_angle>6.280000</max_angle>
+                </horizontal>
+            </scan>
+            <range>
+                <min>0.120000</min>
+                <max>3.5</max>
+                <resolution>0.015000</resolution>
+            </range>
+            <noise>
+                <type>gaussian</type>
+                <mean>0.0</mean>
+                <stddev>0.01</stddev>
+            </noise>
             </ray>
-            <plugin name="laser_controller" filename="libgazebo_ros_ray_sensor.so">
-                <ros>
-                    <argument>--remap ~/out:=scan</argument>
-                </ros>
+            <plugin filename="libgazebo_ros_ray_sensor.so" name="lidar_plugin">
+                <topic_name>scan</topic_name>
                 <output_type>sensor_msgs/LaserScan</output_type>
-                <!-- Changed to match link name -->
                 <frame_name>lidar_link</frame_name>
             </plugin>

File: project_ws/src/telerobot_description/urdf/robot_base.xacro (robot description, xacro)
@@ -3,12 +3,12 @@
     <!-- Robot Base-->
     <xacro:property name="base_length" value="0.6" />
-    <xacro:property name="base_width" value="0.6" />
+    <xacro:property name="base_width" value="0.4" />
     <xacro:property name="base_height" value="0.2" />
     <xacro:property name="wheel_radius" value="0.1" />
     <xacro:property name="wheel_length" value="0.05" />
     <!-- tower-->
-    <xacro:property name="tower_length" value="0.3" />
-    <xacro:property name="tower_width" value="0.3" />
-    <xacro:property name="tower_height" value="1.0" />
+    <xacro:property name="tower_length" value="0.2" />
+    <xacro:property name="tower_width" value="0.2" />
+    <xacro:property name="tower_height" value="0.7" />
     <link name="base_footprint" />
     <link name="base_link">

File: project_ws/src/telerobot_description/urdf/robot_base_gazebo.xacro (robot description, xacro)
@@ -1,26 +1,69 @@
-ä<?xml version="1.0"?>
-<robot xmlns:xacro="http://www.ros.org/wiki/xacro"
-      xmlns:ros_gz_sim="http://gazebosim.org/schema/ros_gz_sim">
+<?xml version="1.0"?>
+<robot xmlns:xacro="http://www.ros.org/wiki/xacro">
+    <gazebo reference="base_link">
+        <material>Gazebo/Blue</material>
+    </gazebo>
+    <gazebo reference="right_wheel_link">
+        <material>Gazebo/Grey</material>
+    </gazebo>
+    <gazebo reference="left_wheel_link">
+        <material>Gazebo/Grey</material>
+    </gazebo>
     <gazebo reference="caster_wheel_link">
+        <material>Gazebo/Grey</material>
         <mu1 value="0.1" />
         <mu2 value="0.1" />
     </gazebo>
     <gazebo>
-        <plugin filename="gz-sim-diff-drive-system"
-                name="gz::sim::systems::DiffDrive">
+        <plugin name="diff_drive_controller" filename="libgazebo_ros_diff_drive.so">
+            <!-- Update rate in Hz -->
+            <update_rate>50</update_rate>
+            <!-- wheels -->
             <left_joint>base_left_wheel_joint</left_joint>
             <right_joint>base_right_wheel_joint</right_joint>
+            <!-- kinematics -->
             <wheel_separation>0.45</wheel_separation>
-            <wheel_radius>0.1</wheel_radius>
-            <frame_id>odom</frame_id>
-            <child_frame_id>base_footprint</child_frame_id>
+            <wheel_diameter>0.2</wheel_diameter>
+            <!-- output -->
+            <publish_odom>true</publish_odom>
+            <publish_odom_tf>true</publish_odom_tf>
+            <publish_wheel_tf>true</publish_wheel_tf>
+            <odometry_topic>odom</odometry_topic>
+            <odometry_frame>odom</odometry_frame>
+            <robot_base_frame>base_footprint</robot_base_frame>
         </plugin>
     </gazebo>
-    <gazebo>
-        <plugin filename="libignition-gazebo6-joint-state-publisher-system"
-                name="gz::sim::systems::JointStatePublisher">
-            <joint_name>base_left_wheel_joint</joint_name>
-            <joint_name>base_right_wheel_joint</joint_name>
+    <link name="imu_link">
+        <inertial>
+            <mass value="0.01" />
+            <inertia ixx="0.0001" ixy="0.0" ixz="0.0"
+                    iyy="0.0001" iyz="0.0"
+                    izz="0.0001" />
+        </inertial>
+    </link>
+    <joint name="imu_joint" type="fixed">
+        <parent link="base_link" />  <!-- Hier den passenden Parent-Link Ihres Roboters eintragen -->
+        <child link="imu_link" />
+        <origin xyz="0.1 0 0.05" rpy="0 0 0" />  <!-- Position und Ausrichtung der IMU anpassen -->
+    </joint>
+    <gazebo reference="imu_link">
+        <gravity>true</gravity>
+        <sensor name="imu_sensor" type="imu">
+        <always_on>true</always_on>
+        <update_rate>100</update_rate>
+        <visualize>true</visualize>
+        <topic>__default_topic__</topic>
+        <plugin filename="libgazebo_ros_imu_sensor.so" name="imu_plugin">
+            <topicName>imu</topicName>
+            <bodyName>imu_link</bodyName>
+            <updateRateHZ>10.0</updateRateHZ>
+            <gaussianNoise>0.0</gaussianNoise>
+            <xyzOffset>0 0 0</xyzOffset>
+            <rpyOffset>0 0 0</rpyOffset>
+            <frameName>imu_link</frameName>
+            <initialOrientationAsReference>false</initialOrientationAsReference>
         </plugin>
+        <pose>0 0 0 0 0 0</pose>
+        </sensor>
     </gazebo>
 </robot>
