Commit message: streamer with asyncio

File: project_ws/install/telerobot_description/share/telerobot_description/urdf/simple_distance.xacro (robot description, xacro)
@@ -1 +1,168 @@
-/media/ros/fedora/home/maylis/Dokumente/TeleNav/project_ws/src/telerobot_description/urdf/simple_distance.xacro
+<?xml version="1.0"?>
+<robot xmlns:xacro="http://www.ros.org/wiki/xacro">
+    <!-- Corrected property names and more reasonable dimensions -->
+    <xacro:property name="lidar_radius" value="0.01" />
+    <xacro:property name="lidar_length" value="0.01" />
+    <link name="tower_distance_link">
+        <visual>
+            <geometry>
+                <cylinder radius="${lidar_radius}" length="${lidar_length}"/>
+            </geometry>
+            <material name="grey" />
+        </visual>
+        <collision>
+            <geometry>
+                <cylinder radius="${lidar_radius}" length="${lidar_length}"/>
+            </geometry>
+        </collision>
+        <xacro:cylinder_inertia m="0.1" r="${lidar_radius}" h="${lidar_length}"
+                           xyz="0 0 0" rpy="0 0 0" />
+    </link>
+    <joint name="base_lidar_joint" type="fixed">
+        <parent link="tower_link" />
+        <child link="tower_distance_link" />
+        <!-- Placing lidar on top of the base (base_height is 0.2) -->
+        <origin xyz="${tower_width/2.0+lidar_length} 0 ${(tower_height*0.5)}" rpy="0 0 0" />
+    </joint>
+    <gazebo reference="tower_distance_link">
+    <sensor name="lidar" type="ray">
+        <always_on>true</always_on>
+        <visualize>true</visualize>
+        <update_rate>1</update_rate>
+        <ray>
+            <scan>
+                <horizontal>
+                    <samples>1</samples>
+                    <resolution>1.0</resolution>
+                    <min_angle>0.0</min_angle>
+                    <max_angle>0.0</max_angle>
+                </horizontal>
+            </scan>
+            <range>
+                <min>0.12</min>
+                <max>3.5</max>
+                <resolution>0.015</resolution>
+            </range>
+            <noise>
+                <type>gaussian</type>
+                <mean>0.0</mean>
+                <stddev>0.01</stddev>
+            </noise>
+        </ray>
+        <plugin filename="libgazebo_ros_ray_sensor.so" name="distance_front">
+            <topic_name>front_distance</topic_name>
+            <output_type>sensor_msgs/Range</output_type>
+            <frame_name>tower_distance_link</frame_name>
+            <radiation_type>infrared</radiation_type>
+        </plugin>
+    </sensor>
+</gazebo>
+    <link name="bumper_distance_front_link">
+        <visual>
+            <geometry>
+                <cylinder radius="${lidar_radius}" length="${lidar_length}"/>
+            </geometry>
+            <material name="grey" />
+        </visual>
+        <collision>
+            <geometry>
+                <cylinder radius="${lidar_radius}" length="${lidar_length}"/>
+            </geometry>
+        </collision>
+        <xacro:cylinder_inertia m="0.1" r="${lidar_radius}" h="${lidar_length}"
+                           xyz="0 0 0" rpy="0 0 0" />
+    </link>
+    <joint name="lower_lidar_joint" type="fixed">
+        <parent link="front_bumper_link" />
+        <child link="bumper_distance_front_link" />
+        <!-- Placing lidar on top of the base (base_height is 0.2) -->
+        <origin xyz="${base_width/2.0+lidar_length} 0 ${(base_height/2.0)}" rpy="0 0 0" />
+    </joint>
+    <gazebo reference="bumper_distance_front_link">
+    <sensor name="lower_lidar" type="ray">
+        <always_on>true</always_on>
+        <visualize>true</visualize>
+        <update_rate>1</update_rate>
+        <ray>
+            <scan>
+                <horizontal>
+                    <samples>1</samples>
+                    <resolution>1.0</resolution>
+                    <min_angle>0.0</min_angle>
+                    <max_angle>0.0</max_angle>
+                </horizontal>
+            </scan>
+            <range>
+                <min>0.12</min>
+                <max>3.5</max>
+                <resolution>0.015</resolution>
+            </range>
+            <noise>
+                <type>gaussian</type>
+                <mean>0.0</mean>
+                <stddev>0.01</stddev>
+            </noise>
+        </ray>
+        <plugin filename="libgazebo_ros_ray_sensor.so" name="distance_lower">
+            <topic_name>lower_distance</topic_name>
+            <output_type>sensor_msgs/Range</output_type>
+            <frame_name>bumper_distance_front_link</frame_name>
+            <radiation_type>infrared</radiation_type>
+        </plugin>
+    </sensor>
+</gazebo>
+    <link name="bumper_distance_back_link">
+        <visual>
+            <geometry>
+                <cylinder radius="${lidar_radius}" length="${lidar_length}"/>
+            </geometry>
+            <material name="grey" />
+        </visual>
+        <collision>
+            <geometry>
+                <cylinder radius="${lidar_radius}" length="${lidar_length}"/>
+            </geometry>
+        </collision>
+        <xacro:cylinder_inertia m="0.1" r="${lidar_radius}" h="${lidar_length}"
+                           xyz="0 0 0" rpy="0 0 0" />
+    </link>
+    <joint name="lower_back_lidar_joint" type="fixed">
+        <parent link="back_bumper_link" />
+        <child link="bumper_distance_back_link" />
+        <!-- Placing lidar on top of the base (base_height is 0.2) -->
+        <origin xyz="${-base_width/2.0-lidar_length} 0 ${(base_height/2.0)}" rpy="0 0 0" />
+    </joint>
+    <gazebo reference="bumper_distance_back_link">
+    <sensor name="lower_back_lidar" type="ray">
+        <always_on>true</always_on>
+        <visualize>true</visualize>
+        <update_rate>1</update_rate>
+        <ray>
+            <scan>
+                <horizontal>
+                    <samples>1</samples>
+                    <resolution>1.0</resolution>
+                    <min_angle>0.0</min_angle>
+                    <max_angle>0.0</max_angle>
+                </horizontal>
+            </scan>
+            <range>
+                <min>0.12</min>
+                <max>3.5</max>
+                <resolution>0.015</resolution>
+            </range>
+            <noise>
+                <type>gaussian</type>
+                <mean>0.0</mean>
+                <stddev>0.01</stddev>
+            </noise>
+        </ray>
+        <plugin filename="libgazebo_ros_ray_sensor.so" name="distance_back">
+            <topic_name>back_distance</topic_name>
+            <output_type>sensor_msgs/Range</output_type>
+            <frame_name>bumper_distance_back_link</frame_name>
+            <radiation_type>infrared</radiation_type>
+        </plugin>
+    </sensor>
+</gazebo>
+</robot>

File: project_ws/install/telerobot_description/share/telerobot_description/urdf/simple_robot.urdf.xacro (robot description, xacro)
@@ -1 +1,101 @@
-/media/ros/fedora/home/maylis/Dokumente/TeleNav/project_ws/src/telerobot_description/urdf/simple_robot.urdf.xacro
+<?xml version="1.0"?>
+<robot name="simple_robo" xmlns:xacro="http://www.ros.org/wiki/xacro">
+    <!-- Robot Base-->
+    <xacro:include filename="common_properties.xacro" />
+    <xacro:include filename="robot_base.xacro" />
+    <gazebo>
+        <plugin name="back_bumper_controller" filename="libgazebo_ros_bumper.so">
+            <alwaysOn>true</alwaysOn>
+            <updateRate>10.0</updateRate>
+            <bumperTopicName>back_bumper</bumperTopicName>
+            <frameName>back_bumper_link</frameName>
+        </plugin>
+    </gazebo>
+    <gazebo>
+        <plugin name="front_bumper_controller" filename="libgazebo_ros_bumper.so">
+            <alwaysOn>true</alwaysOn>
+            <updateRate>10.0</updateRate>
+            <bumperTopicName>front_bumper</bumperTopicName>
+            <frameName>front_bumper_link</frameName>
+        </plugin>
+    </gazebo>
+    <gazebo reference="base_link">
+        <material>Gazebo/Blue</material>
+    </gazebo>
+    <gazebo reference="right_wheel_link">
+        <material>Gazebo/Grey</material>
+    </gazebo>
+    <gazebo reference="left_wheel_link">
+        <material>Gazebo/Grey</material>
+    </gazebo>
+    <gazebo reference="caster_wheel_link">
+        <material>Gazebo/Grey</material>
+        <mu1 value="0.1" />
+        <mu2 value="0.1" />
+    </gazebo>
+    <gazebo>
+        <plugin name="diff_drive" filename="libgazebo_ros_diff_drive.so">
+            <!-- Update rate in Hz -->
+            <update_rate>50</update_rate>
+            <!-- wheels -->
+            <left_joint>base_left_wheel_joint</left_joint>
+            <right_joint>base_right_wheel_joint</right_joint>
+            <!-- kinematics -->
+            <wheel_separation>0.45</wheel_separation>
+            <wheel_diameter>0.2</wheel_diameter>
+            <!-- output -->
+            <publish_odom>true</publish_odom>
+            <publish_odom_tf>true</publish_odom_tf>
+            <publish_wheel_tf>true</publish_wheel_tf>
+            <odometry_topic>odom</odometry_topic>
+            <odometry_frame>odom</odometry_frame>
+            <robot_base_frame>base_footprint</robot_base_frame>
+        </plugin>
+    </gazebo>
+    <!-- Sensors-->
+    <xacro:property name="camera_length" value="0.01" />
+    <xacro:property name="camera_width" value="0.1" />
+    <xacro:property name="camera_height" value="0.05" />
+    <link name="camera_link">
+        <visual>
+            <geometry>
+                <box size="${camera_length} ${camera_width} ${camera_height}" />
+            </geometry>
+            <material name="grey" />
+        </visual>
+        <collision>
+            <geometry>
+                <box size="${camera_length} ${camera_width} ${camera_height}" />
+            </geometry>
+        </collision>
+        <xacro:box_inertia m="0.1" l="${camera_length}" w="${camera_width}" h="${camera_height}"
+                           xyz="0 0 0" rpy="0 0 0" />
+    </link>
+    <joint name="base_camera_joint" type="fixed">
+        <parent link="tower_link" />
+        <child link="camera_link" />
+        <origin xyz="${(tower_width + camera_length) / 2.0} 0 ${tower_height * 0.8}" rpy="0 0 0" />
+    </joint>
+    <link name="camera_link_optical">
+    </link>
+    <joint name="camera_optical_joint" type="fixed">
+        <!-- these values have to be these values otherwise the gazebo camera
+            image won't be aligned properly with the frame it is supposedly
+            originating from -->
+        <origin xyz="0 0 0" rpy="${-pi/2} 0 ${-pi/2}"/>
+        <parent link="camera_link"/>
+        <child link="camera_link_optical"/>
+    </joint>
+    <gazebo reference="camera_link">
+        <material>Gazebo/Red</material>
+        <sensor name="camera_sensor" type="camera">
+            <pose>0 0 0 0 0 0</pose>
+            <visualize>true</visualize>
+            <update_rate>10.0</update_rate>
+            <plugin name="front_robot" filename="libgazebo_ros_camera.so">
+                <frame_name>camera_link_optical</frame_name>
+            </plugin>
+        </sensor>
+    </gazebo>
+    <xacro:include filename="simple_distance.xacro"/>
+</robot>

File: project_ws/src/telerobot_description/urdf/simple_distance.xacro (robot description, xacro)
@@ -4,5 +4,5 @@
     <xacro:property name="lidar_radius" value="0.01" />
     <xacro:property name="lidar_length" value="0.01" />
-    <link name="lidar_link">
+    <link name="tower_distance_link">
         <visual>
             <geometry>
@@ -21,55 +21,13 @@
     <joint name="base_lidar_joint" type="fixed">
         <parent link="tower_link" />
-        <child link="lidar_link" />
+        <child link="tower_distance_link" />
         <!-- Placing lidar on top of the base (base_height is 0.2) -->
         <origin xyz="${tower_width/2.0+lidar_length} 0 ${(tower_height*0.5)}" rpy="0 0 0" />
     </joint>
-    <link name="lower_lidar_link">
-        <visual>
-            <geometry>
-                <cylinder radius="${lidar_radius}" length="${lidar_length}"/>
-            </geometry>
-            <material name="grey" />
-        </visual>
-        <collision>
-            <geometry>
-                <cylinder radius="${lidar_radius}" length="${lidar_length}"/>
-            </geometry>
-        </collision>
-        <xacro:cylinder_inertia m="0.1" r="${lidar_radius}" h="${lidar_length}"
-                           xyz="0 0 0" rpy="0 0 0" />
-    </link>
-    <joint name="lower_lidar_joint" type="fixed">
-        <parent link="front_bumper_link" />
-        <child link="lower_lidar_link" />
-        <!-- Placing lidar on top of the base (base_height is 0.2) -->
-        <origin xyz="${base_width/2.0+lidar_length} 0 ${(base_height/2.0)}" rpy="0 0 0" />
-    </joint>
-    <link name="lower_back_lidar_link">
-        <visual>
-            <geometry>
-                <cylinder radius="${lidar_radius}" length="${lidar_length}"/>
-            </geometry>
-            <material name="grey" />
-        </visual>
-        <collision>
-            <geometry>
-                <cylinder radius="${lidar_radius}" length="${lidar_length}"/>
-            </geometry>
-        </collision>
-        <xacro:cylinder_inertia m="0.1" r="${lidar_radius}" h="${lidar_length}"
-                           xyz="0 0 0" rpy="0 0 0" />
-    </link>
-    <joint name="lower_back_lidar_joint" type="fixed">
-        <parent link="back_bumper_link" />
-        <child link="lower_back_lidar_link" />
-        <!-- Placing lidar on top of the base (base_height is 0.2) -->
-        <origin xyz="${-base_width/2.0-lidar_length} 0 ${(base_height/2.0)}" rpy="0 0 0" />
-    </joint>
-   <gazebo reference="lidar_link">
+    <gazebo reference="tower_distance_link">
     <sensor name="lidar" type="ray">
         <always_on>true</always_on>
         <visualize>true</visualize>
-        <update_rate>5</update_rate>
+        <update_rate>1</update_rate>
         <ray>
             <scan>
@@ -95,14 +53,35 @@
             <topic_name>front_distance</topic_name>
             <output_type>sensor_msgs/Range</output_type>
-            <frame_name>lidar_link</frame_name>
+            <frame_name>tower_distance_link</frame_name>
             <radiation_type>infrared</radiation_type>
         </plugin>
     </sensor>
 </gazebo>
-<gazebo reference="lower_lidar_link">
+    <link name="bumper_distance_front_link">
+        <visual>
+            <geometry>
+                <cylinder radius="${lidar_radius}" length="${lidar_length}"/>
+            </geometry>
+            <material name="grey" />
+        </visual>
+        <collision>
+            <geometry>
+                <cylinder radius="${lidar_radius}" length="${lidar_length}"/>
+            </geometry>
+        </collision>
+        <xacro:cylinder_inertia m="0.1" r="${lidar_radius}" h="${lidar_length}"
+                           xyz="0 0 0" rpy="0 0 0" />
+    </link>
+    <joint name="lower_lidar_joint" type="fixed">
+        <parent link="front_bumper_link" />
+        <child link="bumper_distance_front_link" />
+        <!-- Placing lidar on top of the base (base_height is 0.2) -->
+        <origin xyz="${base_width/2.0+lidar_length} 0 ${(base_height/2.0)}" rpy="0 0 0" />
+    </joint>
+    <gazebo reference="bumper_distance_front_link">
     <sensor name="lower_lidar" type="ray">
         <always_on>true</always_on>
         <visualize>true</visualize>
-        <update_rate>5</update_rate>
+        <update_rate>1</update_rate>
         <ray>
             <scan>
@@ -128,14 +107,35 @@
             <topic_name>lower_distance</topic_name>
             <output_type>sensor_msgs/Range</output_type>
-            <frame_name>lower_lidar_link</frame_name>
+            <frame_name>bumper_distance_front_link</frame_name>
             <radiation_type>infrared</radiation_type>
         </plugin>
     </sensor>
 </gazebo>
-<gazebo reference="lower_back_lidar_link">
+    <link name="bumper_distance_back_link">
+        <visual>
+            <geometry>
+                <cylinder radius="${lidar_radius}" length="${lidar_length}"/>
+            </geometry>
+            <material name="grey" />
+        </visual>
+        <collision>
+            <geometry>
+                <cylinder radius="${lidar_radius}" length="${lidar_length}"/>
+            </geometry>
+        </collision>
+        <xacro:cylinder_inertia m="0.1" r="${lidar_radius}" h="${lidar_length}"
+                           xyz="0 0 0" rpy="0 0 0" />
+    </link>
+    <joint name="lower_back_lidar_joint" type="fixed">
+        <parent link="back_bumper_link" />
+        <child link="bumper_distance_back_link" />
+        <!-- Placing lidar on top of the base (base_height is 0.2) -->
+        <origin xyz="${-base_width/2.0-lidar_length} 0 ${(base_height/2.0)}" rpy="0 0 0" />
+    </joint>
+    <gazebo reference="bumper_distance_back_link">
     <sensor name="lower_back_lidar" type="ray">
         <always_on>true</always_on>
         <visualize>true</visualize>
-        <update_rate>5</update_rate>
+        <update_rate>1</update_rate>
         <ray>
             <scan>
@@ -161,5 +161,5 @@
             <topic_name>back_distance</topic_name>
             <output_type>sensor_msgs/Range</output_type>
-            <frame_name>lower_back_lidar_link</frame_name>
+            <frame_name>bumper_distance_back_link</frame_name>
             <radiation_type>infrared</radiation_type>
         </plugin>
