Commit message: keyboard control

File: project_ws/install/telerobot_description/share/telerobot_description/urdf/common_properties.xacro (robot description, xacro)
@@ -9,4 +9,7 @@
     <material name="red">
         <color rgba="0.5 0 0 1" />
+    </material>
+    <material name="black">
+        <color rgba="0 0 0 1" />
     </material>
     <xacro:macro name="box_inertia" params="m l w h xyz rpy">
@@ -37,3 +40,38 @@
         </inertial>
     </xacro:macro>
+    <xacro:macro name="gazebo_lidar_sensor" params="sensor_name link_name update_rate samples resolution min_angle max_angle min max range_resolution plugin_name topic_name output_type frame_name ">
+        <gazebo reference="${link_name}">
+            <sensor name="${sensor_name}" type="ray">
+                <always_on>true</always_on>
+                <visualize>true</visualize>
+                <update_rate>10</update_rate>
+                <ray>
+                    <scan>
+                        <horizontal>
+                            <samples>${samples}</samples>
+                            <resolution>${resolution}</resolution>
+                            <min_angle>${min_angle}</min_angle>
+                            <max_angle>${max_angle}</max_angle>
+                        </horizontal>
+                    </scan>
+                    <range>
+                        <min>${min}</min>
+                        <max>${max}</max>
+                        <resolution>0.15</resolution>
+                    </range>
+                    <noise>
+                        <type>gaussian</type>
+                        <mean>0.0</mean>
+                        <stddev>0.01</stddev>
+                    </noise>
+                </ray>
+                <plugin filename="libgazebo_ros_ray_sensor.so" name="${plugin_name}">
+                    <topic_name>${topic_name}</topic_name>
+                    <output_type>${output_type}</output_type>
+                    <frame_name>${frame_name}</frame_name>
+                    <radiation_type>infrared</radiation_type>
+                </plugin>
+            </sensor>
+        </gazebo>
+    </xacro:macro>
 </robot>

File: project_ws/install/telerobot_description/share/telerobot_description/urdf/simple_distance.xacro (robot description, xacro)
@@ -41,5 +41,5 @@
             <range>
                 <min>0.12</min>
-                <max>3.5</max>
+                <max>300</max>
                 <resolution>0.015</resolution>
             </range>
@@ -52,5 +52,5 @@
         <plugin filename="libgazebo_ros_ray_sensor.so" name="distance_front">
             <topic_name>front_distance</topic_name>
-            <output_type>sensor_msgs/Range</output_type>
+            <output_type>sensor_msgs/LaserScan</output_type>
             <frame_name>tower_distance_link</frame_name>
             <radiation_type>infrared</radiation_type>
@@ -95,5 +95,5 @@
             <range>
                 <min>0.12</min>
-                <max>3.5</max>
+                <max>300</max>
                 <resolution>0.015</resolution>
             </range>
@@ -134,35 +134,35 @@
     </joint>
     <gazebo reference="bumper_distance_back_link">
-    <sensor name="lower_back_lidar" type="ray">
-        <always_on>true</always_on>
-        <visualize>true</visualize>
-        <update_rate>1</update_rate>
-        <ray>
-            <scan>
-                <horizontal>
-                    <samples>1</samples>
-                    <resolution>1.0</resolution>
-                    <min_angle>0.0</min_angle>
-                    <max_angle>0.0</max_angle>
-                </horizontal>
-            </scan>
-            <range>
-                <min>0.12</min>
-                <max>3.5</max>
-                <resolution>0.015</resolution>
-            </range>
-            <noise>
-                <type>gaussian</type>
-                <mean>0.0</mean>
-                <stddev>0.01</stddev>
-            </noise>
-        </ray>
-        <plugin filename="libgazebo_ros_ray_sensor.so" name="distance_back">
-            <topic_name>back_distance</topic_name>
-            <output_type>sensor_msgs/Range</output_type>
-            <frame_name>bumper_distance_back_link</frame_name>
-            <radiation_type>infrared</radiation_type>
-        </plugin>
-    </sensor>
-</gazebo>
+        <sensor name="lower_back_lidar" type="ray">
+            <always_on>true</always_on>
+            <visualize>true</visualize>
+            <update_rate>1</update_rate>
+            <ray>
+                <scan>
+                    <horizontal>
+                        <samples>1</samples>
+                        <resolution>1.0</resolution>
+                        <min_angle>0.0</min_angle>
+                        <max_angle>0.0</max_angle>
+                    </horizontal>
+                </scan>
+                <range>
+                    <min>0.12</min>
+                    <max>300</max>
+                    <resolution>0.015</resolution>
+                </range>
+                <noise>
+                    <type>gaussian</type>
+                    <mean>0.0</mean>
+                    <stddev>0.01</stddev>
+                </noise>
+            </ray>
+            <plugin filename="libgazebo_ros_ray_sensor.so" name="distance_back">
+                <topic_name>back_distance</topic_name>
+                <output_type>sensor_msgs/Range</output_type>
+                <frame_name>bumper_distance_back_link</frame_name>
+                <radiation_type>infrared</radiation_type>
+            </plugin>
+        </sensor>
+    </gazebo>
 </robot>
